Commit message: 可以在已有地图上生成轨迹，按照规划的路径行动

File: mecanumbot-ros-pkg/description/copy of mecanumbot.urdf (robot description, URDF)
Before this commit: robot mecanumbot, 6 links, 5 joints
Links:
- added link camera_link, mass 0.69591; collision mesh filename=package://mecanumbot/description/camera_link.STL; visual mesh filename=package://mecanumbot/description/camera_link.STL
- added link camera_supports, mass 0.041975; collision mesh filename=package://mecanumbot/description/camera_supports.STL; visual mesh filename=package://mecanumbot/description/camera_supports.STL
- added link e_stop, mass 0.016321; collision mesh filename=package://mecanumbot/description/e_stop.STL; visual mesh filename=package://mecanumbot/description/e_stop.STL
- added link mid_plate_link, mass 0.23689; collision mesh filename=package://mecanumbot/description/mid_plate_link.STL; visual mesh filename=package://mecanumbot/description/mid_plate_link.STL
- added link top_plate_link, mass 0.28331; collision mesh filename=package://mecanumbot/description/top_plate_link.STL; visual mesh filename=package://mecanumbot/description/top_plate_link.STL
- added link top_plate_supports, mass 0.011427; collision mesh filename=package://mecanumbot/description/top_plate_supports.STL; visual mesh filename=package://mecanumbot/description/top_plate_supports.STL
- link base_link: geometry collision mesh filename=package://mecanumbot/description/base_link.STL; visual mesh filename=package://mecanumbot/description/base_link.STL
Joints:
- added joint base_link_to_e_stop: type fixed, parent base_link, child e_stop, origin xyz=0.0184384919793947 0.144923807858542 -0.0836412158001629 rpy=-6.12303176911189E-17 0 0, axis 0 0 0
- added joint base_link_to_mid_plate_link: type fixed, parent base_link, child mid_plate_link, origin xyz=-0.0447365080206053 -0.0182511921414576 -0.0204662158001629 rpy=1.5707963267949 0 0, axis 0 0 0
- added joint camera_supports_to_camera_link: type fixed, parent camera_supports, child camera_link, origin xyz=0.097 0.10242 0.0175000000000002 rpy=-1.5707963267949 -1.5707963267949 0, axis 0 0 0
- added joint mid_plate_link_to_top_plate_supports: type fixed, parent mid_plate_link, child top_plate_supports, origin xyz=-0.0325563676649805 0.015675 0.006161057906821 rpy=1.5707963267949 0 0, axis 0 0 0
- added joint top_plate_link_to_camera_supports: type fixed, parent top_plate_link, child camera_supports, origin xyz=-0.29 -0.097 0 rpy=1.5707963267949 0 1.5707963267949, axis 0 0 0
- added joint top_plate_supports_to_top_plate_link: type fixed, parent top_plate_supports, child top_plate_link, origin xyz=0.0325563676649805 0.163838942093179 -0.015675 rpy=3.14159265358979 -8.67361737988403E-17 1.5707963267949, axis 0 0 0
- joint base_link_to_base_laser: origin xyz=0.3 -0.2 0 rpy=0 -6.12303176911189E-17 -1.5707963267949 -> xyz=-0.0447365080206049 -0.117567277135445 -0.00506621580016293 rpy=0 -6.12303176911189E-17 -1.5707963267949
- joint base_link_to_bl_wheel_joint: origin xyz=-0.25 0.2 -0.1 rpy=0 0 1.5707963267949 -> xyz=0.0788180033333974 0.110748807858542 -0.0851412158001625 rpy=1.5707963267949 0 0
- joint base_link_to_br_wheel_joint: origin xyz=-0.25 -0.2 -0.1 rpy=0 0 -1.5707963267949 -> xyz=-0.168326164695638 0.110748807858543 -0.0851412158001639 rpy=2.07266866801634 0 3.14159265358979
- joint base_link_to_fl_wheel_joint: origin xyz=0.25 0.2 -0.1 rpy=0 0 1.5707963267949 -> xyz=0.0788531486544269 -0.147251192141458 -0.0851412158001636 rpy=1.5707963267949 0 0
- joint base_link_to_fr_wheel_joint: origin xyz=0.25 -0.2 -0.1 rpy=0 0 -1.5707963267949 -> xyz=-0.168291019374608 -0.147251192141458 -0.0851412158001628 rpy=2.08567039686228 0 3.14159265358979
